File: LeapSD-2.0/leapsd.kicad_pcb (KiCad board)
At the start: 2 copper layers, 43.8 x 33.4 mm, 12 parts

Commit message: small tweak
Parts:
- REF**: value IC_FSA642UMX -> FSA642UMX
Changed lines of the file:
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@@
         (effects (font (size 1 1) (thickness 0.15)))
     )
-    (fp_text value "IC_FSA642UMX" (at -2 1) (layer "F.SilkS")
-        (effects (font (size 0.5 0.5) (thickness 0.125)))
+    (fp_text value "FSA642UMX" (at 1.769569 0.113618) (layer "F.SilkS")
+        (effects (font (size 0.4 0.4) (thickness 0.1) bold))
     )
     (fp_circle (center -2 -1) (end -1.9 -1)
